File: KiCAD/Driver/GREG-MTRDRV.kicad_sch (KiCad schematic)
At the start: 85 parts, among them J1 MOTOR1, J2 MOTOR2, J3 MOTOR1, J4 MOTOR2, J5 MOTOR1, J6 MOTOR2, J7 XT60-M, SW1 SW_Push, U1 STM32G474RETx, U2 DRV8262DDWR, U3 DRV8262DDWR, U4 DRV8262DDWR, U5 TPS543B20RVFT, U6 LMR51430, Y1 24MHz

Commit message: Add journal and update readme
Parts:
- removed J7: XT60-M, footprint:AMASS_XT60-M, symbol XT60-M:XT60-M
- added J7: PWR, TerminalBlock_Phoenix:TerminalBlock_Phoenix_MKDS-1,5-2-5.08_1x02_P5.08mm_Horizontal, symbol Connector:Screw_Terminal_01x02
- added J8: Conn_01x02_Pin, 2PinJST:JST_XH_B2B-XH-AM_1x02_P2.50mm_Vertical, symbol Connector:Conn_01x02_Pin
- C12: footprint Capacitor_SMD:C_0402_1005Metric -> Capacitor_SMD:C_0603_1608Metric
- C14, C20, C26: footprint Capacitor_SMD:C_1206_3216Metric -> Capacitor_SMD:C_Elec_6.3x7.7
Connections:
- net +5V is gone; now on net PWR: C15.1, C16.1, C21.1, C22.1, C27.1, C28.1, J1.4 (Pin_4), J2.4 (Pin_4), J3.4 (Pin_4), J4.4 (Pin_4), J5.4 (Pin_4), J6.4 (Pin_4)
- net GNDA is gone; now on net GND: C34.1, C35.2, R17.2, R18.1, R19.1, R20.1, U5.29 (AGND)
- net +3.3V: no longer C12.2, C13.1, C14.1, C18.2, C19.1, C20.1, C24.2, C25.1, C26.1, C29.1, C30.1, C31.1, C32.1, C34.2, C37.1, C38.1, C43.1, U2.11 (VM), U2.12 (VM), U2.2 (VM), U2.21 (VM), U2.25 (VCC/NSLEEP), U3.11 (VM), U3.12 (VM), U3.2 (VM), U3.21 (VM), U3.25 (VCC/NSLEEP), U4.11 (VM), U4.12 (VM), U4.2 (VM), U4.21 (VM), U4.25 (VCC/NSLEEP), U5.21 (PVIN), U5.22 (PVIN), U5.23 (PVIN), U5.24 (PVIN), U5.25 (PVIN), U5.26 (VDD), U6.3 (VIN), U6.5 (EN)
- net CAN_RX: now also J8.2 (Pin_2)
- net CAN_TX: now also J8.1 (Pin_1)
- net GND: now also J7.2 (Pin_2)
- net PWR: now also C12.2, C13.1, C14.1, C18.2, C19.1, C20.1, C24.2, C25.1, C26.1, U2.11 (VM), U2.12 (VM), U2.2 (VM), U2.21 (VM), U3.11 (VM), U3.12 (VM), U3.2 (VM), U3.21 (VM), U4.11 (VM), U4.12 (VM), U4.2 (VM), U4.21 (VM)
- net VCP1: no longer C18.1, C24.1, U2.1 (VCP/GND), U4.1 (VCP/GND)
- removed net CPH1: C11.2, C17.2, C23.2, U2.44 (CPH/GND), U3.44 (CPH/GND), U4.44 (CPH/GND)
- removed net CPL1: C11.1, C17.1, C23.1, U2.43 (CPL/DVDD), U3.43 (CPL/DVDD), U4.43 (CPL/DVDD)
- net DVDD renamed VCC
- net VCC: now also C29.1, C30.1, C31.1, C32.1, C34.2, C37.1, C38.1, C43.1, U2.25 (VCC/NSLEEP), U3.25 (VCC/NSLEEP), U4.25 (VCC/NSLEEP), U5.21 (PVIN), U5.22 (PVIN), U5.23 (PVIN), U5.24 (PVIN), U5.25 (PVIN), U5.26 (VDD), U6.3 (VIN), U6.5 (EN), J7.1 (Pin_1)
- new net C1PH1: C11.2, U3.44 (CPH/GND)
- new net C1PL1: C11.1, U3.43 (CPL/DVDD)
- new net C2PH1: C17.2, U2.44 (CPH/GND)
- new net C2PL1: C17.1, U2.43 (CPL/DVDD)
- new net C3PH1: C23.2, U4.44 (CPH/GND)
- new net C3PL1: C23.1, U4.43 (CPL/DVDD)
- new net VCP2: C18.1, U2.1 (VCP/GND)
- new net VCP3: C24.1, U4.1 (VCP/GND)
