File: KiCAD/SBC/Connectivity.kicad_sch (KiCad schematic)
At the start: 40 parts, among them J1 Micro_SD_Card_Det1, J19 Microphone, J2 RJ45_JK0654219, J3 USB_A_Stacked, J4 USB_C_Receptacle_USB2.0_16P, J5 HDMI_A, J6 Camera 1, J7 AudioJack3, J8 DEBUG, J9 Camera 2, U5 RTL8211EG-VB-CG, U6 SN74CBTLV16292GR, Y1 25MHz

Commit message: Add journal and update readme
Parts:
- J4: footprint USBC:HRO_TYPE-C-31-M-12 -> Connector_USB:USB_C_Receptacle_HRO_TYPE-C-31-M-12
- Y1: footprint Crystal:Crystal_SMD_3225-4Pin_3.2x2.5mm -> Crystal:Crystal_SMD_3215-2Pin_3.2x1.5mm
Connections:
- removed net CT_COMMON: J2.1 (MXCT3), J2.12 (MXCT1), J2.6 (MXCT2), J2.7 (MXCT4)
- no-connect marks 42 -> 47
Changed lines of the file:
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@@
 	)
 	(junction
-		(at 138.43 64.77)
-		(diameter 0)
-		(color 0 0 0 0)
-	)
-	(junction
 		(at 308.61 157.48)
 		(diameter 0)
@@
 	)
 	(junction
-		(at 138.43 69.85)
-		(diameter 0)
-		(color 0 0 0 0)
-	)
-	(junction
 		(at 134.62 92.71)
 		(diameter 0)
@@
 	)
 	(junction
-		(at 138.43 74.93)
-		(diameter 0)
-		(color 0 0 0 0)
-	)
-	(junction
 		(at 52.07 193.04)
 		(diameter 0)
@@
 	)
 	(no_connect
+		(at 146.05 54.61)
+	)
+	(no_connect
 		(at 369.57 59.69)
 	)
@@
 	)
 	(no_connect
+		(at 146.05 74.93)
+	)
+	(no_connect
 		(at 369.57 82.55)
 	)
@@
 	)
 	(no_connect
+		(at 49.53 144.78)
+	)
+	(no_connect
 		(at 410.21 199.39)
 	)
@@
 	)
 	(no_connect
+		(at 146.05 85.09)
+	)
+	(no_connect
 		(at 425.45 120.65)
 	)
@@
 		(at 49.53 86.36)
 	)
+	(no_connect
+		(at 146.05 64.77)
+	)
 	(wire
 		(pts
@@
 	(wire
 		(pts
-			(xy 138.43 64.77) (xy 146.05 64.77)
-		)
-		(stroke
-			(width 0)
-			(type default)
-		)
-	)
-	(wire
-		(pts
 			(xy 410.21 156.21) (xy 420.37 156.21)
 		)
@@
 	(wire
 		(pts
-			(xy 125.73 69.85) (xy 138.43 69.85)
-		)
-		(stroke
-			(width 0)
-			(type default)
-		)
-	)
-	(wire
-		(pts
 			(xy 142.24 151.13) (xy 142.24 154.94)
 		)
@@
 	(wire
 		(pts
-			(xy 146.05 85.09) (xy 138.43 85.09)
-		)
-		(stroke
-			(width 0)
-			(type default)
-		)
-	)
-	(wire
-		(pts
 			(xy 387.35 158.75) (xy 377.19 158.75)
 		)
@@
 	(wire
 		(pts
-			(xy 138.43 74.93) (xy 138.43 69.85)
-		)
-		(stroke
-			(width 0)
-			(type default)
-		)
-	)
-	(wire
-		(pts
 			(xy 231.14 73.66) (xy 229.87 73.66)
 		)
@@
 	(wire
 		(pts
-			(xy 138.43 85.09) (xy 138.43 74.93)
-		)
-		(stroke
-			(width 0)
-			(type default)
-		)
-	)
-	(wire
-		(pts
 			(xy 229.87 73.66) (xy 229.87 72.39)
 		)
@@
 	(wire
 		(pts
-			(xy 138.43 69.85) (xy 138.43 64.77)
-		)
-		(stroke
-			(width 0)
-			(type default)
-		)
-	)
-	(wire
-		(pts
 			(xy 364.49 105.41) (xy 369.57 105.41)
 		)
@@
 	(wire
 		(pts
-			(xy 138.43 64.77) (xy 138.43 54.61)
-		)
-		(stroke
-			(width 0)
-			(type default)
-		)
-	)
-	(wire
-		(pts
 			(xy 293.37 67.31) (xy 298.45 67.31)
 		)
@@
 	(wire
 		(pts
-			(xy 138.43 54.61) (xy 146.05 54.61)
-		)
-		(stroke
-			(width 0)
-			(type default)
-		)
-	)
-	(wire
-		(pts
 			(xy 46.99 129.54) (xy 49.53 129.54)
 		)
@@
 	(wire
 		(pts
-			(xy 138.43 74.93) (xy 146.05 74.93)
-		)
-		(stroke
-			(width 0)
-			(type default)
-		)
-	)
-	(wire
-		(pts
 			(xy 364.49 67.31) (xy 369.57 67.31)
 		)
@@
 		)
 	)
-	(label "CT_COMMON"
-		(at 125.73 69.85 0)
-		(effects
-			(font
-				(size 1.27 1.27)
-			)
-			(justify left bottom)
-		)
-	)
 	(label "C1D6"
 		(at 377.19 184.15 0)
@@
 			)
 		)
-		(property "Footprint" "Crystal:Crystal_SMD_3225-4Pin_3.2x2.5mm"
+		(property "Footprint" "Crystal:Crystal_SMD_3215-2Pin_3.2x1.5mm"
 			(at 186.69 147.32 0)
 			(effects
@@
 			)
 		)
-		(property "Footprint" "USBC:HRO_TYPE-C-31-M-12"
+		(property "Footprint" "Connector_USB:USB_C_Receptacle_HRO_TYPE-C-31-M-12"
 			(at 242.57 68.58 0)
 			(effects
